Commit message: third commit

File: src/urdf/robot.urdf (robot description, URDF)
Before this commit: robot rosweb, 3 links, 0 joints
Links:
- link fr_wheel: mass 0.0 -> 0; geometry collision box size=0 0 0; visual cylinder length=0.0 radius=

Commit message: commit

File: src/urdf/robot.urdf (robot description, URDF)
Before this commit: robot rosweb, 3 links, 0 joints
Links:
- added link bl_wheel, mass 10; collision cylinder length=0.105 radius=0.276; visual cylinder length=0.175 radius=0.276
- added link br_wheel, mass 10; collision cylinder length=0.105 radius=0.276; visual cylinder length=0.105 radius=0.276
- added link fl_wheel, mass 10; collision cylinder length=0.105 radius=0.276; visual cylinder length=0.105 radius=0.276
- link base_footprint: mass 0 -> 0.001; geometry visual box size=0.001 0.001 0.0011
- link base_link: mass 0 -> None
- link fr_wheel: mass 0 -> 10; geometry collision cylinder length=0.105 radius=0.276; visual cylinder length=0.105 radius=0.276
